File: RXBox.kicad_pcb (KiCad board)
At the start: 2 copper layers, 4.5 x 3.5 mm, 76 parts, among them J1 SMA, J2 USB_A, U1 RTL2832U, U2 M24C02-WMN, U3 R820T2, U4 AP2112K-3.3, U5 74AUP1G74, U6 74LVC1G17, U7 USBLC6-2SC6, X1 19.2 MHz

Commit message: started routing
Parts:
- moved R3 1.60 mm to (140.1, 73.1)
- moved U2 1.48 mm to (144.9, 75.1)
- moved R4 1.45 mm to (140.1, 74.4)
- moved C17 1.44 mm to (125.5, 71.3)
- moved C2 1.42 mm to (125.6, 73.9)
- moved C15 1.42 mm to (125.6, 74.8)
- moved L6 1.41 mm to (125.6, 72.6)
- moved L4 1.40 mm to (125.6, 75.8)
- moved R1 1.40 mm to (125.6, 76.8)
- moved L1 1.40 mm to (123.7, 73.2)
- moved L3 1.40 mm to (123.7, 72.0)
- moved C33 1.10 mm to (121.0, 72.3)
- moved C36 0.70 mm to (137.6, 67.7), turned to -90 degrees
- moved C8 0.68 mm to (133.9, 67.0)
- moved R2 0.22 mm to (133.1, 76.7)
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Routing:
- net +1V2: track 0.00 -> 41.9 mm, vias 0 -> 5
- net /TUNER_SCL: track 0.00 -> 18.9 mm, vias 0 -> 2
- net /TUNER_SDA: track 0.00 -> 18.1 mm, vias 0 -> 2
- net VBUS: track 0.00 -> 15.9 mm
- net +3V3: track 0.00 -> 9.59 mm
- net /EEPROM_SCL: track 0.00 -> 9.09 mm
- net /EEPROM_SDA: track 0.00 -> 8.90 mm
- net /RTL_DP: track 0.00 -> 7.80 mm
- net /RTL_DM: track 0.00 -> 7.70 mm
- net /1V2_FILT_1: track 0.00 -> 7.58 mm, vias 0 -> 2
- net /RTL_3V3: track 0.00 -> 6.71 mm
- net Net-(C36-Pad2): track 0.00 -> 5.95 mm
- net Net-(L1-Pad1): track 0.00 -> 5.17 mm
- net Net-(U5-C): track 0.00 -> 4.83 mm
- net Net-(U1-R): track 0.00 -> 4.12 mm
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- added copper zone on B.Cu, net Earth
- added copper zone on F.Cu, net Earth
- added copper zone on In1.Cu, net Earth
- added copper zone on In2.Cu, net Earth
Other:
- board size 4.5 x 3.5 mm -> 60 x 16.9 mm
- copper layers 2 -> 4

Commit message: done?
Parts:
- J1: footprint Connector_Coaxial:MMCX_Molex_73415-0961_Horizontal_1.0mm-PCB -> Connector_Coaxial:SMA_Samtec_SMA-J-P-H-ST-EM1_EdgeMount
- moved J1 1.85 mm to (164.9, 70.2), turned to 0 degrees
- moved C18 0.65 mm to (154.2, 67.2)
- moved C19 0.65 mm to (152.3, 67.2)
- moved C20 0.65 mm to (153.3, 67.2)
- moved C23 0.60 mm to (157.2, 70.8)
- moved R2 0.30 mm to (132.8, 76.7), turned to 90 degrees
- moved R3 0.15 mm to (140.2, 73.1)
- moved R4 0.15 mm to (140.2, 74.4)
Routing:
- net Earth: track 0.00 -> 37.0 mm, vias 0 -> 44
- net /IF_N: track 0.00 -> 31.1 mm, vias 0 -> 2
- net /IF_P: track 0.00 -> 30.0 mm, vias 0 -> 2
- net /RTL_CLK: track 1.64 -> 25.5 mm
- net /RTL_IF_AGC: track 0.00 -> 18.4 mm, vias 0 -> 2
- net +3V3: track 9.59 -> 27.4 mm, vias 0 -> 15
- net +1V2: track 41.9 -> 53.9 mm, vias 5 -> 7
- net Net-(J1-In): track 0.00 -> 6.50 mm
- net Net-(U3-TF2P): track 0.00 -> 4.10 mm
- net Net-(U3-TF1P): track 0.00 -> 3.65 mm
- net /IF_AGC: track 0.00 -> 2.89 mm
- net Net-(U3-CP): track 0.00 -> 2.87 mm
- net /RTL_3V3: track 6.71 -> 9.21 mm, vias 0 -> 4
- net Net-(C29-Pad2): track 0.00 -> 2.33 mm
- net Net-(U3-VDD_PLL): track 0.00 -> 2.31 mm
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- added copper zone on In2.Cu, net +3V3
- added copper zone on In2.Cu, net /RTL_3V3
- removed copper zone on In2.Cu, net Earth
Other:
- board size 60 x 16.9 mm -> 56.6 x 17.8 mm

Commit message: done sdr?!
Parts:
- removed TP1: 28.8MHz, TestPoint:TestPoint_Pad_D1.0mm
- removed TP2: 9.6MHz, TestPoint:TestPoint_Pad_D1.0mm
- removed TP3: 19.2MHz CMOS, TestPoint:TestPoint_Pad_D1.0mm
- added D2: LED, LED_SMD:LED_0603_1608Metric, F.Cu at (122.5, 63.8)
- added R14: 330R, Resistor_SMD:R_0402_1005Metric, F.Cu at (119.9, 63.8)
- moved C35 6.38 mm to (142.3, 63.7), turned to 90 degrees
- moved C21 5.88 mm to (146.1, 70.3)
- moved X1 5.76 mm to (144.1, 70.2)
- moved C36 4.99 mm to (142.1, 69.8), turned to 90 degrees
- moved U6 4.74 mm to (142.9, 66.2), turned to 90 degrees
- moved C34 4.53 mm to (143.8, 63.7)
- moved R13 4.19 mm to (143.4, 68.3), turned to 180 degrees
- moved U5 3.35 mm to (145.3, 65.0), turned to 90 degrees
- moved U2 2.79 mm to (142.2, 74.3)
- moved C1 2.58 mm to (147.2, 64.7)
- moved L13 2.35 mm to (149.2, 70.3)
- moved R4 2.16 mm to (138.1, 74.2), turned to 90 degrees
- moved R3 2.07 mm to (139.7, 71.1), turned to 180 degrees
- moved C5 1.31 mm to (147.8, 69.8), turned to -90 degrees
- moved L11 0.80 mm to (147.7, 66.0), turned to -90 degrees
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Connections:
- net /1V2_FILT_1 renamed /sdr/1V2_FILT_1
- net /1V2_FILT_2 renamed /sdr/1V2_FILT_2
- net /1V2_FILT_3 renamed /sdr/1V2_FILT_3
- net /BAND_PASS renamed /sdr/BAND_PASS
- net /D renamed /sdr/D
- net /EEPROM_SCL renamed /sdr/EEPROM_SCL
- net /EEPROM_SDA renamed /sdr/EEPROM_SDA
- net /IF_AGC renamed /sdr/IF_AGC
- net /IF_I_N renamed /sdr/IF_I_N
- net /IF_I_P renamed /sdr/IF_I_P
- net /IF_N renamed /sdr/IF_N
- net /IF_P renamed /sdr/IF_P
- net /IF_Q_N renamed /sdr/IF_Q_N
- net /IF_Q_P renamed /sdr/IF_Q_P
- net /RTL_3V3 renamed /sdr/RTL_3V3
- net /RTL_CLK renamed /sdr/RTL_CLK
- net /RTL_DM renamed /sdr/RTL_DM
- net /RTL_DP renamed /sdr/RTL_DP
- net /RTL_IF_AGC renamed /sdr/RTL_IF_AGC
- net /TUNER_SCL renamed /sdr/TUNER_SCL
- net /TUNER_SDA renamed /sdr/TUNER_SDA
- net /TUNER_XIN renamed /sdr/TUNER_XIN
Routing:
- net /sdr/RTL_3V3: track 9.21 -> 31.4 mm
- net Earth: track 37.0 -> 31.4 mm, vias 44 -> 122
- net Net-(U5-C): track 4.83 -> 1.18 mm
- net /sdr/EEPROM_SDA: track 10.0 -> 6.47 mm
- net Net-(C36-Pad2): track 5.95 -> 3.01 mm
- net VBUS: track 15.9 -> 13.1 mm
- net /sdr/TUNER_XIN: track 3.72 -> 1.21 mm
- net /sdr/BAND_PASS: track 3.14 -> 0.89 mm
- net /sdr/RTL_CLK: track 25.5 -> 23.5 mm
- net +3V3: track 27.4 -> 25.5 mm, vias 15 -> 16
- net /sdr/EEPROM_SCL: track 9.09 -> 7.81 mm
- net Net-(D2-K): track 0.00 -> 1.25 mm
- net /sdr/TUNER_SCL: track 19.2 -> 18.4 mm
- net /sdr/TUNER_SDA: track 18.1 -> 17.4 mm
- added copper zone on In2.Cu, net (none)
- removed copper zone on In2.Cu, net /sdr/RTL_3V3
Other:
- board text added: "Max Kendall"
- board text added: "RXBox SDR+"

Commit message: lowkey forgot git exists
Routing:
- net Net-(U3-RF_IN): track 1.30 -> 2.60 mm
