File: RXBox.kicad_sch (KiCad schematic)
At the start: 76 parts, among them J1 SMA, J2 USB_A, U1 RTL2832U, U2 M24C02-WMN, U3 R820T2, U4 AP2112K-3.3, U5 74AUP1G74, U6 74LVC1G17, U7 USBLC6-2SC6, X1 19.2 MHz

Commit message: done?
Parts:
- J1: footprint Connector_Coaxial:MMCX_Molex_73415-0961_Horizontal_1.0mm-PCB -> Connector_Coaxial:SMA_Samtec_SMA-J-P-H-ST-EM1_EdgeMount
Changed lines of the file:
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@@
 			)
 		)
-		(property "Footprint" "Connector_Coaxial:MMCX_Molex_73415-0961_Horizontal_1.0mm-PCB"
+		(property "Footprint" "Connector_Coaxial:SMA_Samtec_SMA-J-P-H-ST-EM1_EdgeMount"
 			(at 149.86 26.67 0)
 			(hide yes)

Commit message: revive project
Parts:
- removed C1, C5: 20pF, Capacitor_SMD:C_0402_1005Metric, symbol Device:C_Small
- removed C10, C11, C12, C13, C14, C15, C16, C17, C18, C19, C2, C21, C22, C24, C25, C28, C29, C34, C35, C4, C6, C7: 100nF, Capacitor_SMD:C_0402_1005Metric, symbol Device:C_Small
- removed C20: 1uF, Capacitor_SMD:C_0402_1005Metric, symbol Device:C_Small
- removed C23, C31: 10nF, Capacitor_SMD:C_0402_1005Metric, symbol Device:C_Small
- removed C26: 330pF, Capacitor_SMD:C_0402_1005Metric, symbol Device:C_Small
- removed C27: 6.8nF, Capacitor_SMD:C_0402_1005Metric, symbol Device:C_Small
- removed C3: 1.3nF, Capacitor_SMD:C_0402_1005Metric, symbol Device:C_Small
- removed C30, C32, C33, C8: 10uF, Capacitor_SMD:C_0402_1005Metric, symbol Device:C_Small
- removed C36: 1nF, Capacitor_SMD:C_0402_1005Metric, symbol Device:C_Small
- removed C9: 47uF, Capacitor_SMD:C_0402_1005Metric, symbol Device:C_Small
- removed D1: BAV99, Package_TO_SOT_SMD:SOT-23, symbol Diode:BAV99
- removed J1: SMA, Connector_Coaxial:SMA_Samtec_SMA-J-P-H-ST-EM1_EdgeMount, symbol Connector:Conn_Coaxial
- removed J2: USB_A, Connector_USB:USB_A_Molex_48037-2200_Horizontal, symbol Connector:USB_A
- removed L1, L3, L4, L5, L6, L9: bead, Inductor_SMD:L_0402_1005Metric, symbol Device:L_Small
- removed L10: 8.2nH, Inductor_SMD:L_0402_1005Metric, symbol Device:L_Small
- removed L11, L13: 1.6uH, Inductor_SMD:L_0402_1005Metric, symbol Device:L_Small
- removed L12: 24nH, Inductor_SMD:L_0402_1005Metric, symbol Device:L_Small
- removed L2: 4.7uH, Inductor_SMD:L_0402_1005Metric, symbol Device:L_Small
- removed L7, L8: 150nH, Inductor_SMD:L_0603_1608Metric, symbol Device:L_Small
- removed R1, R10: 10kR, Resistor_SMD:R_0402_1005Metric, symbol Device:R_Small_US
- removed R11, R3, R4, R5, R6: 4.7kR, Resistor_SMD:R_0402_1005Metric, symbol Device:R_Small_US
- removed R12, R13: 100kR, Resistor_SMD:R_0402_1005Metric, symbol Device:R_Small_US
- removed R2: 1M, Resistor_SMD:R_0402_1005Metric, symbol Device:R_Small_US
- removed R7, R8: 220R, Resistor_SMD:R_0402_1005Metric, symbol Device:R_Small_US
- removed R9: 1.8kR, Resistor_SMD:R_0402_1005Metric, symbol Device:R_Small_US
- removed TP1: 28.8MHz, TestPoint:TestPoint_Pad_D1.0mm, symbol Connector:TestPoint
- removed TP2: 9.6MHz, TestPoint:TestPoint_Pad_D1.0mm, symbol Connector:TestPoint
- removed TP3: 19.2MHz CMOS, TestPoint:TestPoint_Pad_D1.0mm, symbol Connector:TestPoint
- removed U1: RTL2832U, Package_DFN_QFN:QFN-48-1EP_6x6mm_P0.4mm_EP4.3x4.3mm_ThermalVias, symbol rtlsdr-symbols:RTL2832U
- removed U2: M24C02-WMN, Package_SO:SOIC-8_3.9x4.9mm_P1.27mm, symbol Memory_EEPROM:M24C02-WMN
- removed U3: R820T2, Package_DFN_QFN:QFN-24-1EP_4x4mm_P0.5mm_EP2.7x2.7mm_ThermalVias, symbol rtlsdr-symbols:R820T2
- removed U4: AP2112K-3.3, Package_TO_SOT_SMD:SOT-23-5, symbol Regulator_Linear:AP2112K-3.3
- removed U5: 74AUP1G74, Package_SON:X2SON-8_1.4x1mm_P0.35mm, symbol 74xGxx:74AUP1G74
- removed U6: 74LVC1G17, Package_TO_SOT_SMD:SOT-353_SC-70-5, symbol 74xGxx:74LVC1G17
- removed U7: USBLC6-2SC6, Package_TO_SOT_SMD:SOT-23-6, symbol Power_Protection:USBLC6-2SC6
- removed X1: 19.2 MHz, Crystal:Crystal_SMD_2016-4Pin_2.0x1.6mm, symbol rtlsdr-symbols:28.8mhz_chinese_tcxo
Connections:
- no-connect marks 15 -> 0
Other:
- added sheet SDR (untitled.kicad_sch)

Commit message: done sdr?!
Parts:
- added D2: LED, LED_SMD:LED_0603_1608Metric, symbol Device:LED
- added R14: 330R, Resistor_SMD:R_0402_1005Metric, symbol Device:R_US
Connections:
- new net: D2.1 (K), R14.1
- new net +3V3: D2.2 (A)
- new net Earth: R14.2
Other:
- removed sheet SDR
- added sheet sdr (sdr.kicad_sch)

Commit message: lowkey forgot git exists
Parts:
- removed D2: LED, LED_SMD:LED_0603_1608Metric, symbol Device:LED
- removed R14: 330R, Resistor_SMD:R_0402_1005Metric, symbol Device:R_US
Other:
- sheet sdr renamed SDR
- added sheet ComputeModule (computemodule.kicad_sch)
- added sheet Interface (interface.kicad_sch)
- added sheet Power (power.kicad_sch)
- added sheet Screen (screen.kicad_sch)
- added sheet Sensors (sensors.kicad_sch)
- sheet SDR ports: added RTL_DM, RTL_DP, SDR_3v3; removed none
- note added: "GPS + IMU (w Magnetometer)"

Commit message: starting to add stuff
Other:
- removed sheet Screen
- sheet ComputeModule ports: added CM_3V3_OUT, CM_5V, HDMI0_CEC, HDMI0_CLK_N, HDMI0_CLK_P, HDMI0_HOTPLUG, HDMI0_SCL, HDMI0_SDA, HDMI0_TX0_N, HDMI0_TX0_P, HDMI0_TX1_N, HDMI0_TX1_P, HDMI0_TX2_N, HDMI0_TX2_P, SCL0, SCL1, SDA0, SDA1, SPI0_CS0, SPI0_CS1, SPI0_MISO, SPI0_MOSI, SPI0_SCLK, UART0_RX, UART0_TX, USB_N, USB_P; removed none
- sheet Interface ports: added LI-ION-, LI-ION-+, LI-ION-TS, USB_D+, USB_D-, USB_PWR_OUT; removed none
- sheet Power ports: added USB_PWR_IN; removed PWR_IN
- note removed: "GPS + IMU (w Magnetometer)"
