File: hardware/rxbox/sbc-power.kicad_sch (KiCad schematic)
At the start: 41 parts, among them U2 SY8088, U3 SY8088, U4 SY8088, U5 SY8088, U6 ME6211C18M5, U7 SY8088

Commit message: finish up journal
Connections:
- net +5V: no longer U2.1 (EN), U3.1 (EN), U4.1 (EN), U5.1 (EN), U6.3 (CE), U7.1 (EN)
- net VCC_DRAM: no longer C17.1, C18.1, L5.2, R9.1
- new net EN_1V8: U5.1 (EN)
- new net EN_AVCC: U6.3 (CE)
- new net EN_CPU: U3.1 (EN)
- new net EN_DRAM: U4.1 (EN)
- new net EN_GEN: U7.1 (EN)
- new net EN_SYS: U2.1 (EN)
- new net VCC_3V3: C17.1, C18.1, L5.2, R9.1
Other:
- added sheet sequencing (sbc-sequencing.kicad_sch)
- note added: "Power Sequencing"
- moved on the sheet: C1, C10, C11, C12, C13, C14, C15, C16, C17, C18, C2, C3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
