File: hardware/rxbox/rxbox.kicad_sch (KiCad schematic)
At the start: 0 parts

Commit message: supervisor + symbol, new journal. jumper for t113 power
Other:
- added sheet dev (dev.kicad_sch)
Changed lines of the file:
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@@
+		)
+	)
+	(sheet
+		(at 172.72 63.5)
+		(size 37.465 24.13)
+		(exclude_from_sim no)
+		(in_bom yes)
+		(on_board yes)
+		(dnp no)
+		(fields_autoplaced yes)
+		(stroke
+			(width 0.1524)
+			(type solid)
+		)
+		(fill
+			(color 0 0 0 0)
+		)
+		(property "Sheetname" "dev"
+			(at 172.72 62.7884 0)
+			(show_name no)
+			(do_not_autoplace no)
+			(effects
+				(font
+					(size 1.27 1.27)
+				)
+				(justify left bottom)
+			)
+		)
+		(property "Sheetfile" "dev.kicad_sch"
+			(at 172.72 88.2146 0)
+			(show_name no)
+			(do_not_autoplace no)
+			(effects
+				(font
+					(size 1.27 1.27)
+				)
+				(justify left top)
+			)
+		)
+		(instances
+			(project "rxbox"
+				(path "/4bda69c0-d40e-4af8-940b-109cd2045912"
+					(page "6")
+				)
+			)
 		)
 	)
