File: hardware/rxbox/ddr3.kicad_sch (KiCad schematic)
At the start: 0 parts

Commit message: draft of ddr circuitry
Parts:
- added C66, C70, C71, C72, C76, C77, C78, C80: 100nF, symbol Device:C_Small
- added C67, C68, C69, C73, C74, C75: 1uF, symbol Device:C_Small
- added C79: 2.2pF, symbol Device:C_Small
- added R63, R64: 2kR, Resistor_SMD:R_0402_1005Metric, symbol Device:R_Small_US
- added R65: 240R, Resistor_SMD:R_0402_1005Metric, symbol Device:R_Small_US
- added R66: 100R, Resistor_SMD:R_0402_1005Metric, symbol Device:R_Small_US
- added U13: (no value), Package_BGA:FBGA-96_7.5x13mm_Layout9x16_P0.8mm, symbol Memory_RAM_Custom:H5TQ4G63EFR
Connections:
- new net: R65.2, U13.L8 (ZQ)
- new net A0: U13.N3 (A0)
- new net A1: U13.P7 (A1)
- new net A10: U13.L7 (A10/AP)
- new net A11: U13.R7 (A11)
- new net A12: U13.N7 (A12/~{BC})
- new net A13: U13.T3 (A13)
- new net A14: U13.T7 (A14)
- new net A2: U13.P3 (A2)
- new net A3: U13.N2 (A3)
- new net A4: U13.P8 (A4)
- new net A5: U13.P2 (A5)
- new net A6: U13.R8 (A6)
- new net A7: U13.R2 (A7)
- new net A8: U13.T8 (A8)
- new net A9: U13.R3 (A9)
- new net BA0: U13.M2 (BA0)
- new net BA1: U13.N8 (BA1)
- new net BA2: U13.M3 (BA2)
- new net CKE: U13.K9 (CKE)
- new net CLK+: C79.1, R66.2, U13.J7 (CK)
- new net CLK-: C79.2, R66.1, U13.K7 (~{CK})
- new net DML: U13.E7 (DML)
- new net DMU: U13.D3 (DMU)
- new net DQL0: U13.E3 (DQL0)
- new net DQL1: U13.F7 (DQL1)
- new net DQL2: U13.F2 (DQL2)
- new net DQL3: U13.F8 (DQL3)
- new net DQL4: U13.H3 (DQL4)
- new net DQL5: U13.H8 (DQL5)
- new net DQL6: U13.G2 (DQL6)
- new net DQL7: U13.H7 (DQL7)
- new net DQSL+: U13.F3 (DQSL)
- new net DQSL-: U13.G3 (~{DQSL})
- new net DQSU+: U13.C7 (DQSU)
- new net DQSU-: U13.B7 (~{DQSU})
- new net DQU0: U13.D7 (DQU0)
- new net DQU1: U13.C3 (DQU1)
- new net DQU2: U13.C8 (DQU2)
- new net DQU3: U13.C2 (DQU3)
- new net DQU4: U13.A7 (DQU4)
- new net DQU5: U13.A2 (DQU5)
- new net DQU6: U13.B8 (DQU6)
- new net DQU7: U13.A3 (DQU7)
- new net Earth: C66.2, C67.2, C68.2, C69.2, C70.2, C71.2, C72.2, C73.2, C74.2, C75.2, C76.2, C77.2, C78.2, C80.2, R64.1, R65.1, U13.A9 (VSS), U13.B1 (VSSQ), U13.B3 (VSS), U13.B9 (VSSQ), U13.D1 (VSSQ), U13.D8 (VSSQ), U13.E1 (VSS), U13.E2 (VSSQ), U13.E8 (VSSQ), U13.F9 (VSSQ), U13.G1 (VSSQ), U13.G8 (VSS), U13.G9 (VSSQ), U13.J2 (VSS), U13.J8 (VSS), U13.M1 (VSS), U13.M9 (VSS), U13.P1 (VSS), U13.P9 (VSS), U13.T1 (VSS), U13.T9 (VSS)
- new net ODT: U13.K1 (ODT)
- new net VCC_DRAM: C67.1, C68.1, C69.1, C70.1, C71.1, C72.1, C73.1, C74.1, C75.1, C76.1, C77.1, C78.1, R63.2, U13.A1 (VDDQ), U13.A8 (VDDQ), U13.B2 (VDD), U13.C1 (VDDQ), U13.C9 (VDDQ), U13.D2 (VDDQ), U13.D9 (VDD), U13.E9 (VDDQ), U13.F1 (VDDQ), U13.G7 (VDD), U13.H2 (VDDQ), U13.H9 (VDDQ), U13.K2 (VDD), U13.K8 (VDD), U13.N1 (VDD), U13.N9 (VDD), U13.R1 (VDD), U13.R9 (VDD)
- new net VREF: C66.1, C80.1, R63.1, R64.2, U13.H1 (VREFDQ), U13.M8 (VREFCA)
- new net ~{CAS}: U13.K3 (~{CAS})
- new net ~{CS}: U13.L2 (~{CS})
- new net ~{RAS}: U13.J3 (~{RAS})
- new net ~{RESET}: U13.T2 (~{RESET})
- new net ~{WE}: U13.L3 (~{WE})
Other:
- note added: "DQ"
- note added: "SYS"
