File: hardware/rxbox/storage.kicad_sch (KiCad schematic)
At the start: 6 parts, among them J2 Micro_SD_Card, U12 GD25QxxxEY

Commit message: draft of ddr circuitry
Parts:
- added C64: 47uF, symbol Device:C_Small
- added R53: 1kR, symbol Device:R_Small_US
- added R55: 10kR, symbol Device:R_Small_US
- added R56: 100kR, symbol Device:R_Small_US
- added R61, R62: 33R, Resistor_SMD:R_0402_1005Metric, symbol Device:R_Small_US
- J2: symbol Connector:Micro_SD_Card -> Connector:Micro_SD_Card_Det1
Connections:
- net Earth: now also J2.6 (VSS), C64.2
- net NOR.SCLK: now also R62.1; no longer U12.6 (SCLK)
- net VCC_3V3: now also J2.4 (VDD), C64.1, R55.2, R56.2
- net D2: now reaches J2.1 (DAT2)
- net D3: now reaches J2.2 (DAT3/CD)
- net CMD: now reaches J2.3 (CMD)
- net CMD: now also R55.1
- net at J2.5 (CLK): now also R61.2
- net D0: now reaches J2.7 (DAT0)
- net D1: now reaches J2.8 (DAT1)
- new net: J2.9 (DET), R53.1, R56.1
- new net: R62.2, U12.6 (SCLK)
- new net CLK: R61.1
- new net DET: R53.2
Other:
- note added: "main boot media"
- moved on the sheet: C62, R50, R51, R52, U12
