File: hardware/rxbox/t113.kicad_sch (KiCad schematic)
At the start: 1 part, among them U1 T113-I

Commit message: finish hooking up wifi+bt, and power
Parts:
- added C36, C53, C54, C55, C56, C57: 100nF, symbol Device:C_Small
- added C37, C38, C42, C43, C48, C50: 10uF, symbol Device:C_Small
- added C39, C40, C41, C44, C45, C46, C47, C51, C52: 2.2uF, symbol Device:C_Small
- added C49: 470nF, symbol Device:C_Small
- added C58, C59: 18pF, symbol Device:C_Small
- added C60, C61: 15pF, symbol Device:C_Small
- added D4: 1N4007, Diode_THT:D_DO-41_SOD81_P10.16mm_Horizontal, symbol Diode:1N4007
- added R33, R34, R36, R37, R39, R40, R41, R47, R49: 0R, Resistor_SMD:R_0402_1005Metric, symbol Device:R_Small_US
- added R38: NC, Resistor_SMD:R_0402_1005Metric, symbol Device:R_Small_US
- added R48: 1MR, Resistor_SMD:R_0402_1005Metric, symbol Device:R_Small_US
- added unit 8 of U1
- added Y2: 24Mhz, Crystal:Crystal_SMD_2016-4Pin_2.0x1.6mm, symbol Device:Crystal_GND24
- added Y3: 32.768kHz, Crystal:Crystal_SMD_3215-2Pin_3.2x1.5mm, symbol Device:Crystal
Connections:
- net CPU_PWM: now also R33.1
- net Earth: now also C37.1, C38.1, C39.1, C40.1, C41.1, C42.1, C43.1, C44.1, C45.1, C46.1, C50.1, C51.1, C52.1, C53.2, C54.1, C55.1, C56.1, C57.1, C58.1, C59.1, C60.1, C61.1, Y2.2 (G), Y2.4 (G)
- net VDD_1V8: now also U1.J4 (VCC-EFUSE), U1.J5 (VCC-PLL), U1.K5 (VCC-RTC), C54.2, C55.2, C56.2, R38.2, R39.2
- net VDD_CPU: now also C37.2, C38.2, C39.2, C40.2, C41.2
- net VDD_SYS: now also C42.2, C43.2, C44.2, C45.2, C46.2; no longer U1.G13 (VDD_SYS)
- net WL_HOST_WAKE: now reaches U1.C6 (PG10)
- net WL_REG_ON: now reaches U1.D5 (PG12)
- net BT_WAKE: now reaches U1.D6 (PG13)
- net BT_HOST_WAKE: now reaches U1.E6 (PG14)
- net at U1.E7 (PG17): now also R41.1
- net BT_RST_N: now reaches U1.F6 (PG15)
- net at U1.Y18 (PD22): now also R33.2
- new net: R36.2, U1.G13 (VDD_SYS)
- new net: R40.1, U1.C19 (ALDO)
- new net: C61.2, R48.2, R49.1, Y3.2
- new net: D4.2 (A), R37.2
- new net: C58.2, R47.1, Y2.3
- new net 1V8_REG: R38.1
- new net 32KHZ: R41.2
- new net AVCC: C47.2, R40.2, U1.C18 (AVCC)
- new net DXIN: C59.2, U1.K1 (DXIN), Y2.1
- new net DXOUT: R47.2, U1.K2 (DXOUT)
- new net GNDA: C47.1, C48.1, C49.1, U1.D18 (AGND)
- new net LDOA-OUT: C51.2, R39.1, U1.L7 (LDOA-OUT)
- new net LDOB-OUT: C52.2, U1.N7 (LDOB-OUT)
- new net LDO_IN: C50.2, D4.1 (K), U1.M7 (LDO-IN)
- new net SYS_FB: R36.1
- new net VCC_3V3: C53.1, C57.2, R37.1, U1.E4 (VCC-PG), U1.G17 (VCC-IO)
- new net VRA1: C48.2, U1.B19 (VRA1)
- new net VRA2: C49.2, U1.B18 (VRA2)
- new net X32KIN: C60.2, R48.1, U1.L2 (X32KIN), Y3.1
- new net X32KOUT: R49.2, U1.L3 (X32KOUT)
- no-connect marks 12 -> 0
Other:
- note added: "int/ext 1v8 int default"
- note added: "probably not the best way to organize decoupling, but oh well"

Commit message: start boot media circuitry
Changed lines of the file:
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@@
 		)
 		(pin "C2"
+			(alternate "SDC0-D1")
 		)
 		(pin "C1"
+			(alternate "SDC0-D0")
 		)
 		(pin "G3"
@@
 		)
 		(pin "E2"
+			(alternate "SDC0-D2")
 		)
 		(pin "P9"
@@
 		)
 		(pin "D1"
+			(alternate "SDC0-CMD")
 		)
 		(pin "L10"
@@
 		)
 		(pin "E3"
+			(alternate "SDC0-D3")
 		)
 		(pin "H19"
@@
 		)
 		(pin "D2"
+			(alternate "SDC0-CLK")
 		)
 		(pin "U20"

Commit message: draft of ddr circuitry
Parts:
- added C63, C65, C81, C82, C83, C84, C85, C86, C87, C88: 100nF, symbol Device:C_Small
- added R54, R57, R58, R59: 0R, Resistor_SMD:R_0402_1005Metric, symbol Device:R_Small_US
- added R67: 240R, Resistor_SMD:R_0402_1005Metric, symbol Device:R_Small_US
Connections:
- net Earth: now also C63.2, C65.2, C81.2, C82.2, C83.2, C84.2, C85.2, C86.2, C87.2, C88.2, R58.2, R67.1
- net VCC_3V3: now also U1.F4 (VCC-PF), U1.G4 (VCC-PC), C63.1, C65.1, R59.2
- net VDD_1V8: now also U1.P14 (VDD18-DRAM), C88.1
- net SDBOOT.D0: now reaches U1.C1 (PF1)
- net SDBOOT.D1: now reaches U1.C2 (PF0)
- net SDBOOT.CMD: now reaches U1.D1 (PF3)
- net SDBOOT.CLK: now reaches U1.D2 (PF2)
- net SDBOOT.DET: now reaches U1.D3 (PF6)
- net SDBOOT.D2: now reaches U1.E2 (PF5)
- net SDBOOT.D3: now reaches U1.E3 (PF4)
- net at U1.F5 (PC5): now also R57.2, R59.1
- net NOR.~{CS}: now reaches U1.G2 (PC3)
- net NOR.SCLK: now reaches U1.G3 (PC2)
- net NOR.HOLD: now reaches U1.G5 (PC7)
- net NOR.WP: now reaches U1.G6 (PC6)
- net at U1.H3 (PC4): now also R54.2, R58.1
- net VCC_DRAM: now reaches U1.N10 (VCC-DRAM)
- net VCC_DRAM: now also U1.N8 (VCC-DRAM), U1.N9 (VCC-DRAM), U1.P10 (VCC-DRAM), U1.P8 (VCC-DRAM), U1.P9 (VCC-DRAM), C82.1, C83.1, C84.1, C85.1, C86.1, C87.1
- net ~{CS}: now reaches U1.R12 (SCS0)
- net A13: now reaches U1.R15 (SA13)
- net DQU7: now reaches U1.R6 (SDQ15)
- net DQU5: now reaches U1.R7 (SDQ13)
- net ~{WE}: now reaches U1.R9 (SWE)
- net CLK+: now reaches U1.T10 (SCKP)
- net ODT: now reaches U1.T12 (SODT0)
- net DQU6: now reaches U1.T4 (SDQ14)
- net DQU3: now reaches U1.T6 (SDQ11)
- net ~{CAS}: now reaches U1.T9 (SCAS)
- net CLK-: now reaches U1.U10 (SCKN)
- net A3: now reaches U1.U13 (SA3)
- net A4: now reaches U1.U15 (SA4)
- net VREF: now reaches U1.U16 (SVREF)
- net VREF: now also C81.1
- net at U1.U17 (SZQ): now also R67.2
- net DQU0: now reaches U1.U4 (SDQ8)
- net DQU2: now reaches U1.U5 (SDQ10)
- net DQU4: now reaches U1.U6 (SDQ12)
- net DQU1: now reaches U1.U7 (SDQ9)
- net ~{RAS}: now reaches U1.U9 (SRAS)
- net BA0: now reaches U1.V10 (SBA0)
- net A5: now reaches U1.V11 (SA5)
- net A0: now reaches U1.V13 (SA0)
- net A2: now reaches U1.V14 (SA2)
- net A14: now reaches U1.V16 (SA14)
- net DQL6: now reaches U1.V5 (SDQ6)
- net DQL1: now reaches U1.V7 (SDQ1)
- net DQL3: now reaches U1.V8 (SDQ3)
- net BA1: now reaches U1.W10 (SBA1)
- net A6: now reaches U1.W11 (SA6)
- net A10: now reaches U1.W12 (SA10)
- net A1: now reaches U1.W13 (SA1)
- net A8: now reaches U1.W14 (SA8)
- net A11: now reaches U1.W15 (SA11)
- net A12: now reaches U1.W16 (SA12)
- net DMU: now reaches U1.W2 (SDQM1)
- net DQSU+: now reaches U1.W3 (SDQS1P)
- net DQL4: now reaches U1.W4 (SDQ4)
- net DQL7: now reaches U1.W5 (SDQ7)
- net DQSL+: now reaches U1.W6 (SDQS0P)
- net DQL0: now reaches U1.W7 (SDQ0)
- net DQL2: now reaches U1.W8 (SDQ2)
- net CKE: now reaches U1.W9 (SCKE0)
- net BA2: now reaches U1.Y11 (SBA2)
- net A7: now reaches U1.Y13 (SA7)
- net A9: now reaches U1.Y15 (SA9)
- net ~{RESET}: now reaches U1.Y17 (SRST)
- net DQSU-: now reaches U1.Y3 (SDQS1N)
- net DQL5: now reaches U1.Y4 (SDQ5)
- net DQSL-: now reaches U1.Y6 (SDQS0N)
- net DML: now reaches U1.Y8 (SDQM0)
- new net NOR.MISO: R57.1
- new net NOR.MOSI: R54.1
- no-connect marks 0 -> 4
Other:
- note added: "naive, change for routing"
- moved on the sheet: C53, C58, C59, C60, C61, R33, R41, R47, R48, R49, U1A, U1B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
